Commit message: nao_description: add (empty) visualization macros for elbow_yaw and fingers

File: nao_description/urdf/nao_robot_structure.urdf.xacro (robot description, xacro)
@@ -81,4 +81,5 @@
       <inertia ixx="0"  ixy="0"  ixz="0" iyy="0" iyz="0" izz="0" />
     </inertial>
+    <xacro:insert_visualization_elbow_yaw side="${side}"/>
   </link>
   <link name = "${side}ElbowRoll_link">
@@ -98,5 +99,7 @@
     <xacro:insert_visualization_wrist side="${side}"/>
   </link>
-  <link name="${side}Hand_link" />
+  <link name="${side}Hand_link">
+    <xacro:insert_visualization_fingers side="${side}"/>
+  </link>
   </xacro:macro>
   <xacro:arm_links side="L" reflect="-1"/>

File: nao_description/urdf/visuals.xacro (robot description, xacro)
@@ -112,3 +112,7 @@
     <xacro:macro name="insert_visualization_cameraBottom" params="">
     </xacro:macro>
+    <xacro:macro name="insert_visualization_fingers" params="side">
+    </xacro:macro>
+    <xacro:macro name="insert_visualization_elbow_yaw" params="side">
+    </xacro:macro>
 </robot>
