Commit message: added mimic tag to RHipYawPitch

File: nao_description/urdf/nao_robot_v3_structure.urdf.xacro (robot description, xacro)
@@ -254,12 +254,20 @@
   <xacro:arm_joints side="R" reflect="1"/>
   <!-- Leg joints -->
+  <joint name="LHipYawPitch" type="revolute">
+    <parent link="Torso_link"/>
+    <child link="LHipYawPitch_link"/>
+    <origin xyz="0 0.05 -0.085" rpy="0 0 0"/>
+    <axis xyz="0 0.707106 -0.707106"/>
+    <limit velocity="3.0" effort="30" lower="-1.145303" upper="0.740810"/>
+  </joint>
+  <joint name="RHipYawPitch" type="revolute">
+    <parent link="Torso_link"/>
+    <child link="RHipYawPitch_link"/>
+    <origin xyz="0 -0.05 -0.085" rpy="0 0 0"/>
+    <axis xyz="0 0.707106 0.707106"/>
+    <limit velocity="3.0" effort="30" lower="-1.145303" upper="0.740810"/>
+    <mimic joint="LHipYawPitch" multiplier="1" offset="0"/>
+  </joint>
   <xacro:macro name="leg_joints" params="side reflect">
-  <joint name="${side}HipYawPitch" type="revolute">
-    <parent link="Torso_link"/>
-    <child link="${side}HipYawPitch_link"/>
-    <origin xyz="0 ${reflect*-0.05} -0.085" rpy="0 0 0"/>
-    <axis xyz="0 0.707106 ${reflect*(0.707106)}"/>
-    <limit velocity="3.0" effort="30" lower="-1.145303" upper="0.740810"/>
-  </joint>
   <joint name="${side}HipPitch" type="revolute">
     <parent link="${side}HipRoll_link"/>

File: nao_description/urdf/nao_robot_v4_structure.urdf.xacro (robot description, xacro)
@@ -266,12 +266,20 @@
   <xacro:arm_joints side="R" reflect="1"/>
   <!-- Leg joints -->
+  <joint name="LHipYawPitch" type="revolute">
+    <parent link="Torso_link"/>
+    <child link="LHipYawPitch_link"/>
+    <origin xyz="0 0.05 -0.085" rpy="0 0 0"/>
+    <axis xyz="0 0.707106 -0.707106"/>
+    <limit velocity="3.0" effort="30" lower="-1.145303" upper="0.740810"/>
+  </joint>
+  <joint name="RHipYawPitch" type="revolute">
+    <parent link="Torso_link"/>
+    <child link="RHipYawPitch_link"/>
+    <origin xyz="0 -0.05 -0.085" rpy="0 0 0"/>
+    <axis xyz="0 0.707106 0.707106"/>
+    <limit velocity="3.0" effort="30" lower="-1.145303" upper="0.740810"/>
+    <mimic joint="LHipYawPitch" multiplier="1" offset="0"/>
+  </joint>
   <xacro:macro name="leg_joints" params="side reflect">
-  <joint name="${side}HipYawPitch" type="revolute">
-    <parent link="Torso_link"/>
-    <child link="${side}HipYawPitch_link"/>
-    <origin xyz="0 ${reflect*-0.05} -0.085" rpy="0 0 0"/>
-    <axis xyz="0 0.707106 ${reflect*(0.707106)}"/>
-    <limit velocity="3.0" effort="30" lower="-1.145303" upper="0.740810"/>
-  </joint>
   <joint name="${side}HipPitch" type="revolute">
     <parent link="${side}HipRoll_link"/>

Commit message: nao_common and nao_robot now compatible to REP-120

File: nao_description/urdf/nao_robot_v3_structure.urdf.xacro (robot description, xacro)
@@ -8,5 +8,6 @@
   Authors: Armin Hornung, Stefan Osswald
   Joint names and properties are according to the Nao-documentation of
-  Aldebaran Robotics ("Kinematics 3.2" for Nao V3.2).
+  Aldebaran Robotics ("Kinematics 3.2" for Nao V3.2) and REP-120:
+  http://ros.org/reps/rep-0120.html
   Note that according to the documentation, the joint limits for the left leg
   are different from the corresponding limits for the right leg.
@@ -20,8 +21,8 @@
         Docs say inertial matrix is in link frame, URDF expects CoM frame
 -->
-  <!-- dummy first link, directly connects with Torso_link -->
+  <!-- dummy first link, directly connects with torso -->
   <link name="base_link" />
   <!-- first real link of the robot, inertial reference frame -->
-  <link name="Torso_link" >
+  <link name="torso" >
   <!--<inertial>
       <origin xyz="0 0 0" rpy="0 0 0"/>
@@ -52,4 +53,5 @@
     <xacro:insert_visualization_head/>
   </link>
+  <link name="gaze" />
   <link name="CameraTop_frame">
     <xacro:insert_visualization_cameraTop/>
@@ -99,8 +101,13 @@
     <xacro:insert_visualization_wrist side="${side}"/>
   </link>
-  <link name="${side}Hand_link">
-    <xacro:insert_visualization_fingers side="${side}"/>
-  </link>
   </xacro:macro>
+  <link name="l_wrist"/>
+  <link name="r_wrist"/>
+  <link name="l_gripper">
+    <xacro:insert_visualization_fingers side="L"/>
+  </link>
+  <link name="r_gripper">
+    <xacro:insert_visualization_fingers side="R"/>
+  </link>
   <xacro:arm_links side="L" reflect="-1"/>
   <xacro:arm_links side="R" reflect="1"/>
@@ -155,13 +162,18 @@
     <xacro:insert_visualization_ankleRoll side="${side}"/>
   </link>
-  <link name="${side}Foot_link">
-    <xacro:insert_visualization_foot side="${side}"/>
-  </link>
   </xacro:macro>
+  <link name="l_ankle" />
+  <link name="r_ankle" />
+  <link name="l_sole">
+    <xacro:insert_visualization_foot side="L"/>
+  </link>
+  <link name="r_sole">
+    <xacro:insert_visualization_foot side="R"/>
+  </link>
   <xacro:leg_links side="L" reflect="-1"/>
   <xacro:leg_links side="R" reflect="1"/>
 <!--   Joints following below -->
   <joint name="base_joint" type="fixed">
-    <child link="Torso_link"/>
+    <child link="torso"/>
     <parent link="base_link"/>
     <origin xyz="0 0 0" rpy="0 0 0" />
@@ -169,5 +181,5 @@
   <!-- Head joints -->
   <joint name="HeadYaw" type="revolute">
-    <parent link="Torso_link"/>
+    <parent link="torso"/>
     <child link="HeadYaw_link"/>
 	<!-- NeckOffsetZ -->
@@ -183,4 +195,9 @@
     <limit velocity="3.0" effort="30" lower="-0.6720" upper="0.5149" />
   </joint>
+  <joint name="gaze_joint" type="fixed">
+    <parent link="HeadPitch_link"/>
+    <child link="gaze"/>
+    <origin xyz="0.0539 0 0.05" />
+  </joint>
   <joint name="CameraTop" type="fixed">
     <parent link="HeadPitch_link"/>
@@ -197,5 +214,5 @@
   <xacro:macro name="arm_joints" params="side reflect">
   <joint name="${side}ShoulderPitch" type="revolute">
-    <parent link="Torso_link"/>
+    <parent link="torso"/>
     <child link="${side}ShoulderPitch_link"/>
     <origin xyz="0 ${reflect*-0.098} 0.1" rpy="0 0 0"/>
@@ -217,10 +234,25 @@
     <limit velocity="3.0" effort="30" lower="-1.8238" upper="1.8238"/>
   </joint>
-  <joint name="${side}Hand" type="fixed">
-    <parent link="${side}WristYaw_link" />
-    <child link="${side}Hand_link" />
+  </xacro:macro>
+  <joint name="l_wrist_joint" type="fixed">
+    <parent link="LWristYaw_link" />
+    <child link="l_wrist" />
+    <origin xyz="0 0 0" />
+  </joint>
+  <joint name="r_wrist_joint" type="fixed">
+    <parent link="RWristYaw_link" />
+    <child link="r_wrist" />
+    <origin xyz="0 0 0" />
+  </joint>
+  <joint name="l_gripper_joint" type="fixed">
+    <parent link="l_wrist" />
+    <child link="l_gripper" />
     <origin xyz="0.058 0 -0.0159" />
   </joint>
-  </xacro:macro>
+  <joint name="r_gripper_joint" type="fixed">
+    <parent link="r_wrist" />
+    <child link="r_gripper" />
+    <origin xyz="0.058 0 -0.0159" />
+  </joint>
   <joint name="LElbowRoll" type="revolute">
     <parent link="LElbowYaw_link"/>
@@ -255,5 +287,5 @@
   <!-- Leg joints -->
   <joint name="LHipYawPitch" type="revolute">
-    <parent link="Torso_link"/>
+    <parent link="torso"/>
     <child link="LHipYawPitch_link"/>
     <origin xyz="0 0.05 -0.085" rpy="0 0 0"/>
@@ -262,5 +294,5 @@
   </joint>
   <joint name="RHipYawPitch" type="revolute">
-    <parent link="Torso_link"/>
+    <parent link="torso"/>
     <child link="RHipYawPitch_link"/>
     <origin xyz="0 -0.05 -0.085" rpy="0 0 0"/>
@@ -297,9 +329,4 @@
     <limit velocity="3.0" effort="30" lower="-1.186448" upper="0.922747"/>
   </joint>
-  <joint name="${side}Foot" type="fixed">
-  	<parent link="${side}AnkleRoll_link" />
-	<child link="${side}Foot_link" />
-	<origin xyz="0 0 -0.04511" />
-  </joint>
   </xacro:macro>
   <joint name="LHipRoll" type="revolute">
@@ -331,4 +358,24 @@
     <limit velocity="3.0" effort="30" lower="-0.388676" upper="0.785875"/>
   </joint>
+  <joint name="l_ankle_joint" type="fixed">
+    <parent link="LAnkleRoll_link" />
+    <child link="l_ankle" />
+    <origin xyz="0 0 0" />
+  </joint>
+  <joint name="r_ankle_joint" type="fixed">
+    <parent link="RAnkleRoll_link" />
+    <child link="r_ankle" />
+    <origin xyz="0 0 0" />
+  </joint>
+  <joint name="l_sole_joint" type="fixed">
+    <parent link="l_ankle" />
+    <child link="l_sole" />
+    <origin xyz="0 0 -0.04511" />
+  </joint>
+  <joint name="r_sole_joint" type="fixed">
+    <parent link="r_ankle" />
+    <child link="r_sole" />
+    <origin xyz="0 0 -0.04511" />
+  </joint>
   <xacro:leg_joints side="L" reflect="-1"/>
   <xacro:leg_joints side="R" reflect="1"/>

File: nao_description/urdf/nao_robot_v4_structure.urdf.xacro (robot description, xacro)
@@ -8,5 +8,6 @@
   Authors: Armin Hornung, Stefan Osswald, Felix Burget
   Joint names and properties are according to the Nao-documentation of
-  Aldebaran Robotics ("Kinematics 4.0" for Nao V4).
+  Aldebaran Robotics ("Kinematics 4.0" for Nao V4) and REP-120:
+  http://ros.org/reps/rep-0120.html
   Note that according to the documentation, the joint limits for the left leg
   are different from the corresponding limits for the right leg.
@@ -20,8 +21,8 @@
         Docs say inertial matrix is in link frame, URDF expects CoM frame
 -->
-  <!-- dummy first link, directly connects with Torso_link -->
+  <!-- dummy first link, directly connects with torso -->
   <link name="base_link" />
   <!-- first real link of the robot, inertial reference frame -->
-  <link name="Torso_link" >
+  <link name="torso" >
   <!--<inertial>
       <origin xyz="0 0 0" rpy="0 0 0"/>
@@ -52,4 +53,5 @@
     <xacro:insert_visualization_head/>
   </link>
+  <link name="gaze" />
   <link name="CameraTop_frame">
     <xacro:insert_visualization_cameraTop/>
@@ -90,8 +92,13 @@
     <xacro:insert_visualization_wrist side="${side}"/>
   </link>
-  <link name="${side}Hand_link">
-    <xacro:insert_visualization_fingers side="${side}"/>
-  </link>
   </xacro:macro>
+  <link name="l_wrist"/>
+  <link name="r_wrist"/>
+  <link name="l_gripper">
+    <xacro:insert_visualization_fingers side="L"/>
+  </link>
+  <link name="r_gripper">
+    <xacro:insert_visualization_fingers side="R"/>
+  </link>
   <xacro:arm_links side="L" reflect="-1"/>
   <xacro:arm_links side="R" reflect="1"/>
@@ -162,13 +169,18 @@
     <xacro:insert_visualization_ankleRoll side="${side}"/>
   </link>
-  <link name="${side}Foot_link">
-    <xacro:insert_visualization_foot side="${side}"/>
-  </link>
   </xacro:macro>
+  <link name="l_ankle" />
+  <link name="r_ankle" />
+  <link name="l_sole">
+    <xacro:insert_visualization_foot side="L"/>
+  </link>
+  <link name="r_sole">
+    <xacro:insert_visualization_foot side="R"/>
+  </link>
   <xacro:leg_links side="L" reflect="-1"/>
   <xacro:leg_links side="R" reflect="1"/>
 <!--   Joints following below -->
   <joint name="base_joint" type="fixed">
-    <child link="Torso_link"/>
+    <child link="torso"/>
     <parent link="base_link"/>
     <origin xyz="0 0 0" rpy="0 0 0" />
@@ -176,5 +188,5 @@
   <!-- Head joints -->
   <joint name="HeadYaw" type="revolute">
-    <parent link="Torso_link"/>
+    <parent link="torso"/>
     <child link="HeadYaw_link"/>
 	<!-- NeckOffsetZ -->
@@ -190,4 +202,9 @@
     <limit velocity="3.0" effort="30" lower="-0.6720" upper="0.5149" />
   </joint>
+  <joint name="gaze_joint" type="fixed">
+    <parent link="HeadPitch_link"/>
+    <child link="gaze"/>
+    <origin xyz="0.0539 0 0.05" />
+  </joint>
   <joint name="CameraTop" type="fixed">
     <parent link="HeadPitch_link"/>
@@ -205,5 +222,5 @@
   <xacro:macro name="arm_joints" params="side reflect">
   <joint name="${side}ShoulderPitch" type="revolute">
-    <parent link="Torso_link"/>
+    <parent link="torso"/>
     <child link="${side}ShoulderPitch_link"/>
     <origin xyz="0 ${reflect*-0.098} 0.1" rpy="0 0 0"/>
@@ -225,10 +242,25 @@
     <limit velocity="3.0" effort="30" lower="-1.8238" upper="1.8238"/>
   </joint>
-  <joint name="${side}Hand" type="fixed">
-    <parent link="${side}WristYaw_link" />
-    <child link="${side}Hand_link" />
-    <origin xyz="0.05775 0 -0.01231" />
-  </joint>
   </xacro:macro>
+  <joint name="l_wrist_joint" type="fixed">
+    <parent link="LWristYaw_link" />
+    <child link="l_wrist" />
+    <origin xyz="0 0 0" />
+  </joint>
+  <joint name="r_wrist_joint" type="fixed">
+    <parent link="RWristYaw_link" />
+    <child link="r_wrist" />
+    <origin xyz="0 0 0" />
+  </joint>
+  <joint name="l_gripper_joint" type="fixed">
+    <parent link="l_wrist" />
+    <child link="l_gripper" />
+    <origin xyz="0.058 0 -0.0159" />
+  </joint>
+  <joint name="r_gripper_joint" type="fixed">
+    <parent link="r_wrist" />
+    <child link="r_gripper" />
+    <origin xyz="0.058 0 -0.0159" />
+  </joint>
   <joint name="LElbowRoll" type="revolute">
     <parent link="LElbowYaw_link"/>
@@ -237,5 +269,4 @@
     <axis xyz="0 0 1"/>
     <limit velocity="3.0" effort="30" lower="-1.5446" upper="-0.0349"/>
-    <!--<limit velocity="3.0" effort="30" lower="-1.5621" upper="-0.0087"/>-->
   </joint>
   <joint name="RElbowRoll" type="revolute">
@@ -245,5 +276,4 @@
     <axis xyz="0 0 1"/>
     <limit velocity="3.0" effort="30" lower="0.0349" upper="1.5446"/>
-    <!--<limit velocity="3.0" effort="30" lower="0.0087" upper="1.5621"/>-->
   </joint>
   <joint name="LShoulderRoll" type="revolute">
@@ -253,5 +283,4 @@
     <axis xyz="0 0 1"/>
     <limit velocity="3.0" effort="30" lower="-0.3142" upper="1.3265"/>
-    <!--<limit velocity="3.0" effort="30" lower="0.0087" upper="1.6494"/>-->
   </joint>
   <joint name="RShoulderRoll" type="revolute">
@@ -261,5 +290,4 @@
     <axis xyz="0 0 1"/>
     <limit velocity="3.0" effort="30" lower="-1.3265" upper="0.3142"/>
-    <!-- <limit velocity="3.0" effort="30" lower="-1.6494" upper="-0.0087"/>-->
   </joint>
   <xacro:arm_joints side="L" reflect="-1"/>
@@ -267,5 +295,5 @@
   <!-- Leg joints -->
   <joint name="LHipYawPitch" type="revolute">
-    <parent link="Torso_link"/>
+    <parent link="torso"/>
     <child link="LHipYawPitch_link"/>
     <origin xyz="0 0.05 -0.085" rpy="0 0 0"/>
@@ -274,5 +302,5 @@
   </joint>
   <joint name="RHipYawPitch" type="revolute">
-    <parent link="Torso_link"/>
+    <parent link="torso"/>
     <child link="RHipYawPitch_link"/>
     <origin xyz="0 -0.05 -0.085" rpy="0 0 0"/>
@@ -310,9 +338,4 @@
     <limit velocity="3.0" effort="30" lower="-1.186448" upper="0.922747"/>
   </joint>
-  <joint name="${side}Foot" type="fixed">
-  	<parent link="${side}AnkleRoll_link" />
-	<child link="${side}Foot_link" />
-	<origin xyz="0 0 -0.04519" />
-  </joint>
   </xacro:macro>
   <joint name="LHipRoll" type="revolute">
@@ -344,4 +367,24 @@
     <limit velocity="3.0" effort="30" lower="-0.388676" upper="0.785875"/>
   </joint>
+  <joint name="l_ankle_joint" type="fixed">
+    <parent link="LAnkleRoll_link" />
+    <child link="l_ankle" />
+    <origin xyz="0 0 0" />
+  </joint>
+  <joint name="r_ankle_joint" type="fixed">
+    <parent link="RAnkleRoll_link" />
+    <child link="r_ankle" />
+    <origin xyz="0 0 0" />
+  </joint>
+  <joint name="l_sole_joint" type="fixed">
+    <parent link="l_ankle" />
+    <child link="l_sole" />
+    <origin xyz="0 0 -0.04519" />
+  </joint>
+  <joint name="r_sole_joint" type="fixed">
+    <parent link="r_ankle" />
+    <child link="r_sole" />
+    <origin xyz="0 0 -0.04519" />
+  </joint>
   <xacro:leg_joints side="L" reflect="-1"/>
   <xacro:leg_joints side="R" reflect="1"/>
